File: arduino.kicad_pcb (KiCad board)
At the start: 2 copper layers, 50.8 x 70.6 mm, 30 parts, among them J1 Conn_01x08_Pin, J10 Conn_01x06_Socket, J12 Conn_01x03_Pin, J2 Conn_01x10_Socket, J3 Barrel_Jack_Switch, J4 Conn_01x02_Socket, J5 Conn_01x06_Socket, J8 Conn_01x08_Pin, SW1 SW_Push, U1 ATmega328-P, U2 L7805, U3 LM317_TO-220, Y1 Crystal

Commit message: Add files via upload
Parts:
- moved SW1 119.2 mm to (250.2, 58.7)
- moved J12 103.7 mm to (241.8, 121.9)
- moved C7 96.5 mm to (254.6, 122.4)
- moved R4 87.5 mm to (240.5, 116.8)
- moved R2 87.4 mm to (240.5, 109.1)
- moved R3 87.3 mm to (240.5, 112.2)
- moved R1 87.3 mm to (240.5, 105.6)
- moved R6 83.7 mm to (237.0, 117.3), turned to 180 degrees
- moved C3 80.4 mm to (234.2, 111.3)
- moved C5 80.0 mm to (220.5, 114.8)
- moved C4 76.1 mm to (227.1, 119.9), turned to -90 degrees
- moved C1 74.9 mm to (220.0, 97.5)
- moved C8 71.4 mm to (224.0, 90.7), turned to 90 degrees
- moved C6 69.3 mm to (217.4, 101.9), turned to -90 degrees
- moved C9 65.3 mm to (218.4, 76.0), turned to -90 degrees
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Routing:
- net GND: track 0.00 -> 219.9 mm
- net VCC: track 0.00 -> 141.5 mm
- net RST: track 0.00 -> 85.9 mm
- net VIN: track 0.00 -> 81.9 mm
- net TX: track 0.00 -> 73.0 mm
- net RX: track 0.00 -> 71.3 mm
- net D13: track 0.00 -> 67.9 mm
- net 3.3: track 0.00 -> 57.5 mm
- net Net-(D2-A): track 0.00 -> 36.0 mm
- net 5V: track 0.00 -> 31.0 mm
- net D10: track 0.00 -> 29.5 mm
- net D8: track 0.00 -> 29.5 mm
- net D12: track 0.00 -> 29.0 mm
- net D9: track 0.00 -> 28.6 mm
- net D11: track 0.00 -> 28.0 mm
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
Commit message: Add files via upload
Parts:
- moved C4 71.8 mm to (233.5, 48.4), turned to 0 degrees
- moved C7 70.6 mm to (233.8, 54.9)
- moved C3 69.4 mm to (233.5, 41.8)
- moved C5 66.2 mm to (218.0, 48.7)
- moved J2 63.8 mm to (214.1, 40.9), turned to 0 degrees
- moved J5 60.5 mm to (240.4, 40.9)
- moved C1 57.0 mm to (218.0, 40.6)
- moved D1 54.3 mm to (239.7, 58.0), turned to 0 degrees
- moved J12 51.5 mm to (203.2, 87.8)
- moved J3 51.4 mm to (231.0, 68.2), turned to 0 degrees
- moved SW1 50.9 mm to (203.0, 77.7)
- moved U2 50.4 mm to (236.8, 66.8)
- moved C6 49.2 mm to (218.0, 52.7), turned to 0 degrees
- moved J8 43.1 mm to (229.1, 40.9)
- moved C2 38.0 mm to (218.0, 44.6), turned to 0 degrees
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Routing:
- net GND: track 219.9 -> 0.00 mm
- net VCC: track 141.5 -> 0.00 mm
- net RST: track 85.9 -> 0.00 mm
- net VIN: track 81.9 -> 0.00 mm
- net TX: track 73.0 -> 0.00 mm
- net RX: track 71.3 -> 0.00 mm
- net D13: track 67.9 -> 0.00 mm
- net 3.3: track 57.5 -> 0.00 mm
- net Net-(D2-A): track 36.0 -> 0.00 mm
- net 5V: track 31.0 -> 0.00 mm
- net D10: track 29.5 -> 0.00 mm
- net D8: track 29.5 -> 0.00 mm
- net D12: track 29.0 -> 0.00 mm
- net D9: track 28.6 -> 0.00 mm
- net D11: track 28.0 -> 0.00 mm
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Other:
- board outline removed

Commit message: Add files via upload
Parts:
- moved R1 126.5 mm to (92.2, 90.9)
- moved C3 126.2 mm to (108.6, 59.4)
- moved C4 126.2 mm to (108.6, 65.9)
- moved C7 126.2 mm to (108.8, 72.5)
- moved J12 126.2 mm to (78.3, 105.4)
- moved J4 126.2 mm to (117.4, 102.9)
- moved J8 126.2 mm to (104.1, 58.4)
- moved R2 126.2 mm to (93.0, 97.8)
- moved R3 126.2 mm to (93.0, 100.9)
- moved R4 126.2 mm to (93.0, 104.0)
- moved R6 126.2 mm to (93.0, 107.2)
- moved SW1 126.2 mm to (78.0, 95.3)
- moved U3 126.2 mm to (111.8, 90.3)
- moved C1 126.2 mm to (93.1, 58.1)
- moved C2 126.2 mm to (93.1, 62.2)
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Connections:
- J1 pad 6: D5 -> GND
- U1 pad 11: D5 -> GND
Routing:
- net GND: track 0.00 -> 150.0 mm, vias 0 -> 1
- net VCC: track 0.00 -> 88.0 mm, vias 0 -> 2
- net D13: track 0.00 -> 61.9 mm
- net D12: track 0.00 -> 55.7 mm
- net D11: track 0.00 -> 49.3 mm
- net D10: track 0.00 -> 43.1 mm
- net D9: track 0.00 -> 35.6 mm
- net D6: track 0.00 -> 25.5 mm
- net D7: track 0.00 -> 24.9 mm
- net D8: track 0.00 -> 21.2 mm
- net TX: track 0.00 -> 18.3 mm
- net RX: track 0.00 -> 18.3 mm
- net D4: track 0.00 -> 18.3 mm
- net D3: track 0.00 -> 18.3 mm
- net D2: track 0.00 -> 18.3 mm
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
Commit message: Add files via upload
Parts:
- moved J8 90.9 mm to (191.0, 85.1), turned to 90 degrees
- moved SW1 75.9 mm to (153.7, 101.3)
- moved J1 34.7 mm to (168.1, 126.2)
- moved J2 34.7 mm to (191.5, 126.2)
- moved C8 34.7 mm to (188.2, 116.6)
- moved J12 34.7 mm to (49.3, 86.3)
- moved J4 34.7 mm to (88.4, 83.8)
- moved C1 34.7 mm to (64.1, 39.1)
- moved C2 34.7 mm to (64.1, 43.1)
- moved C3 34.7 mm to (79.6, 40.3)
- moved C4 34.7 mm to (79.6, 46.9)
- moved C5 34.7 mm to (64.1, 47.2)
- moved C6 34.7 mm to (64.1, 51.2)
- moved C7 34.7 mm to (79.9, 53.4)
- moved D2 34.7 mm to (75.6, 77.8)
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Connections:
- J1 pad 6: GND -> D5
- J8 pad 6: RST -> DTR
- R3 pad 2: RST -> DTR
- SW1 pad 1: RST -> DTR
- U1 pad 1: RST -> DTR
- U1 pad 11: GND -> D5
Routing:
- net 3.3: track 0.00 -> 83.5 mm
- net VCC: track 88.0 -> 166.7 mm
- net DTR: track 0.00 -> 70.3 mm
- net D5: track 0.00 -> 26.7 mm
- net GND: track 150.0 -> 146.2 mm
- net D12: track 55.7 -> 53.2 mm
- net D11: track 49.3 -> 47.5 mm
- net D13: track 61.9 -> 60.2 mm
- net D10: track 43.1 -> 41.7 mm

Commit message: Add files via upload
Parts:
- moved R4 215.7 mm to (274.1, 35.8), turned to -90 degrees
- moved R3 214.2 mm to (270.0, 23.1), turned to 180 degrees
- moved R6 213.4 mm to (270.9, 35.8), turned to -90 degrees
- moved C5 212.7 mm to (275.9, 27.2)
- moved C6 212.7 mm to (275.9, 31.2)
- moved C1 206.5 mm to (270.3, 27.2)
- moved C2 206.5 mm to (270.3, 31.2)
- moved D2 195.6 mm to (270.3, 58.2)
- moved D3 189.0 mm to (270.3, 51.1)
- moved C4 185.9 mm to (265.2, 36.4)
- moved C7 185.9 mm to (265.5, 42.9)
- moved C3 185.7 mm to (265.0, 28.7)
- moved D1 179.9 mm to (265.4, 47.2), turned to -90 degrees
- moved R1 156.2 mm to (209.3, 16.5)
- moved R2 155.0 mm to (206.0, 16.5), turned to 180 degrees
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Connections:
- J3 pad 1: Net-(D1-A) -> VIN
Routing:
- net GND: track 146.2 -> 310.8 mm, vias 1 -> 6
- net VIN: track 0.00 -> 161.4 mm, vias 0 -> 1
- net 5V: track 0.00 -> 104.9 mm
- net VCC: track 166.7 -> 236.1 mm, vias 2 -> 4
- net 3.3: track 83.5 -> 128.3 mm, vias 0 -> 2
- net DTR: track 70.3 -> 100.0 mm, vias 0 -> 2
- net D13: track 60.2 -> 84.9 mm, vias 0 -> 1
- net TX: track 18.3 -> 36.4 mm, vias 0 -> 2
- net Net-(U3-ADJ): track 0.00 -> 16.2 mm
- net Net-(D2-A): track 0.00 -> 15.3 mm
- net RX: track 18.3 -> 32.1 mm, vias 0 -> 2
- net Net-(D3-A): track 0.00 -> 8.40 mm
- net 5VU: track 0.00 -> 4.74 mm
Other:
- board outline added: 90 x 60 mm

Commit message: Add files via upload
Parts:
- moved J4 54.1 mm to (162.1, 86.8)
- moved C1 54.1 mm to (220.8, 49.2)
- moved C2 54.1 mm to (220.8, 53.3)
- moved C8 54.1 mm to (188.8, 76.9)
- moved D1 54.1 mm to (216.0, 69.3)
- moved J1 54.1 mm to (168.7, 86.5)
- moved J12 54.1 mm to (148.4, 79.8)
- moved J2 54.1 mm to (192.1, 86.5)
- moved J3 54.1 mm to (158.0, 52.5)
- moved J5 54.1 mm to (158.1, 71.8)
- moved J8 54.1 mm to (191.6, 45.4)
- moved R1 54.1 mm to (159.8, 38.5)
- moved R2 54.1 mm to (156.5, 38.5)
- moved R3 54.1 mm to (220.5, 45.1)
- moved R6 54.1 mm to (221.5, 57.8)
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Routing:
- net DTR: track 100.0 -> 100.5 mm
Other:
- board text added: "SOUPTIK"

Commit message: Add files via upload
Routing:
- net VIN: track 161.4 -> 205.8 mm
- net DTR: track 100.5 -> 106.0 mm
- net VCC: track 236.1 -> 233.7 mm
- net Net-(D2-A): track 15.3 -> 17.3 mm
- net 3.3: track 128.1 -> 130.0 mm
- net 5V: track 104.9 -> 106.6 mm, vias 0 -> 2
- net D13: track 84.9 -> 86.1 mm
- net RX: track 32.1 -> 33.0 mm
- net GND: track 310.8 -> 311.5 mm
